File: Temp Reader/Temp Reader.kicad_pcb (KiCad board)
At the start: 2 copper layers, 3 parts, among them U1 ESP32-C3-DevKitM-1, U2 DHT11, U4 NRF24L01_Breakout

Commit message: 2.First Schematic Look
No Buck

Raw schematic
Parts:
- U1: value ESP32-C3-DevKitM-1 -> ESP32-WROOM-32; footprint RF_Module:ESP32-C3-DevKitM-1 -> RF_Module:ESP32-WROOM-32
- U2: value DHT11 -> BME280; footprint Sensor:Aosong_DHT11_5.5x12.0_P2.54mm -> Package_LGA:Bosch_LGA-8_2.5x2.5mm_P0.65mm_ClockwisePinNumbering
- moved U2 72.9 mm to (34.6, 116.2)
- moved U1 68.7 mm to (56.9, 102.9)
Connections:
- U1 pad 1: Net-(U1-GND-Pad1) -> GND
- U1 pad 10: unconnected-(U1-IO1-Pad10) -> /CE
- U1 pad 11: unconnected-(U1-IO10-Pad11) -> /IRQ
- U1 pad 12: Net-(U1-GND-Pad1) -> /CSB
- U1 pad 13: Net-(U1-5V-Pad13) -> unconnected-(U1-IO14-Pad13)
- U1 pad 14: Net-(U1-5V-Pad13) -> unconnected-(U1-IO12-Pad14)
- U1 pad 15: Net-(U1-GND-Pad1) -> GND
- U1 pad 16: Net-(U1-GND-Pad1) -> unconnected-(U1-IO13-Pad16)
- U1 pad 19: Net-(U1-GND-Pad1) -> unconnected-(U1-SCS/CMD-Pad19)
- U1 pad 2: Net-(U1-3V3-Pad2) -> +3.3V
- U1 pad 24: Net-(U1-GND-Pad1) -> unconnected-(U1-IO2-Pad24)
- U1 pad 27: Net-(U1-GND-Pad1) -> unconnected-(U1-IO16-Pad27)
- U1 pad 3: Net-(U1-3V3-Pad2) -> unconnected-(U1-EN-Pad3)
- U1 pad 30: Net-(U1-GND-Pad1) -> /SCK
- U1 pad 6: Net-(U1-GND-Pad1) -> unconnected-(U1-IO34-Pad6)
- U1 pad 8: Net-(U1-GND-Pad1) -> unconnected-(U1-IO32-Pad8)
- U2 pad 1: unconnected-(U2-VDD-Pad1) -> GND
- U2 pad 2: unconnected-(U2-DATA-Pad2) -> /IO27
- U2 pad 3: unconnected-(U2-NC-Pad3) -> /IO23
- U2 pad 4: unconnected-(U2-GND-Pad4) -> /IO18
- U4 pad 1: unconnected-(U4-GND-Pad1) -> GND
- U4 pad 2: unconnected-(U4-VCC-Pad2) -> +3.3V
- U4 pad 3: unconnected-(U4-CE-Pad3) -> /IO25
- U4 pad 4: unconnected-(U4-~{CSN}-Pad4) -> /IO22
- U4 pad 5: unconnected-(U4-SCK-Pad5) -> /IO18
- U4 pad 6: unconnected-(U4-MOSI-Pad6) -> /IO23
- U4 pad 7: unconnected-(U4-MISO-Pad7) -> /IO19
- U4 pad 8: unconnected-(U4-IRQ-Pad8) -> /IO26

Commit message: **First PCB , Not done yet
Parts:
- added C1: 100nF, Capacitor_SMD:C_0201_0603Metric, F.Cu at (156.5, 48.1)
- added C10: 22uF, Capacitor_SMD:C_1206_3216Metric, F.Cu at (160.6, 70.4)
- added C2: 100nF, Capacitor_SMD:C_0201_0603Metric, F.Cu at (156.5, 49.9)
- added C3: 100nF, Capacitor_SMD:C_0201_0603Metric, F.Cu at (183.8, 67.5)
- added C4: 10uF, Capacitor_SMD:C_1206_3216Metric, F.Cu at (182.3, 67.5)
- added C5: 100nF, Capacitor_SMD:C_0201_0603Metric, F.Cu at (163.6, 41.3)
- added C6: 10uF, Capacitor_SMD:C_1206_3216Metric, F.Cu at (161.5, 41.2)
- added C7: 22uF, Capacitor_SMD:C_1206_3216Metric, F.Cu at (160.6, 68.0)
- added C8: 22uF, Capacitor_SMD:C_1206_3216Metric, F.Cu at (160.5, 54.7)
- added C9: 100nF, Capacitor_SMD:C_0201_0603Metric, F.Cu at (161.6, 61.2)
- added L1: 2.2 uH, Inductor_SMD:L_Bourns-SRN4018, F.Cu at (160.7, 64.2)
- added R1: 31.25k, Resistor_SMD:R_0201_0603Metric, F.Cu at (158.0, 61.1)
- added R2: 10k, Resistor_SMD:R_0201_0603Metric, F.Cu at (158.0, 59.5)
- added R3: 100k, Resistor_SMD:R_0201_0603Metric, F.Cu at (158.9, 56.3)
- added R4: 10k, Resistor_SMD:R_0201_0603Metric, F.Cu at (163.6, 43.4)
- added U5: AP62150WU, Package_TO_SOT_SMD:TSOT-23-6, F.Cu at (160.2, 58.7)
- moved U2 141.4 mm to (159.0, 48.9), turned to -90 degrees
- moved U1 129.0 mm to (173.8, 48.6)
- moved U4 120.6 mm to (186.5, 68.6), turned to 90 degrees
Connections:
- U1 pad 10: /CE -> /IO25
- U1 pad 11: /IRQ -> /IO26
- U1 pad 12: /CSB -> /IO27
- U1 pad 3: unconnected-(U1-EN-Pad3) -> Net-(U1-EN)
- U1 pad 30: /SCK -> /IO18
- U1 pad 31: /MISO -> /IO19
- U1 pad 36: /CSN -> /IO22
- U1 pad 37: /MOSI -> /IO23
Routing:
- net +3.3V: track 0.00 -> 88.9 mm, vias 0 -> 3
- net /IO23: track 0.00 -> 54.1 mm, vias 0 -> 2
- net /IO19: track 0.00 -> 51.6 mm, vias 0 -> 2
- net /IO18: track 0.00 -> 47.3 mm, vias 0 -> 2
- net /IO26: track 0.00 -> 34.4 mm
- net /IO25: track 0.00 -> 30.9 mm, vias 0 -> 1
- net /IO22: track 0.00 -> 25.8 mm, vias 0 -> 1
- net /IO27: track 0.00 -> 9.68 mm
- net Net-(U5-SW): track 0.00 -> 6.80 mm
- net Net-(U5-EN): track 0.00 -> 4.62 mm
- net Vin: track 0.00 -> 2.99 mm
- net Net-(U5-FB): track 0.00 -> 2.16 mm
- net Net-(U1-EN): track 0.00 -> 1.63 mm
- net Net-(U5-BST): track 0.00 -> 1.39 mm
- added copper zone on F.Cu, net GND
