File: Temp Reader/Temp Reader.kicad_pcb (KiCad board)
At the start: 2 copper layers, 19 parts, among them U1 ESP32-WROOM-32, U2 BME280, U4 NRF24L01_Breakout, U5 AP62150WU

Commit message: 1.1.1
Parts:
- added C11: 100nF, Capacitor_SMD:C_0201_0603Metric, F.Cu at (79.9, 126.3)
- added C12: 10uF, Capacitor_SMD:C_1206_3216Metric, F.Cu at (75.8, 127.1)
- added C15: 100nF, Capacitor_SMD:C_0201_0603Metric, F.Cu at (79.9, 128.0)
- added C16: 10uF, Capacitor_SMD:C_1206_3216Metric, F.Cu at (75.8, 130.4)
- added C17: 22uF, Capacitor_SMD:C_1206_3216Metric, F.Cu at (75.8, 133.8)
- added C18: 100nF, Capacitor_SMD:C_0201_0603Metric, F.Cu at (79.9, 129.8)
- added C19: 22uF, Capacitor_SMD:C_1206_3216Metric, F.Cu at (75.8, 137.1)
- added C20: 22uF, Capacitor_SMD:C_1206_3216Metric, F.Cu at (75.8, 140.5)
- added J1: DisplayConnetor, Connector_PinSocket_1.27mm:PinSocket_1x08_P1.27mm_Vertical, F.Cu at (83.7, 108.9)
- added L2: 2.2 uH, Inductor_SMD:L_Bourns-SRN4018, F.Cu at (88.7, 128.2)
- added R5: 10k, Resistor_SMD:R_0201_0603Metric, F.Cu at (79.9, 131.5)
- added R6: 100k, Resistor_SMD:R_0201_0603Metric, F.Cu at (79.9, 133.3)
- added R7: 31.25k, Resistor_SMD:R_0201_0603Metric, F.Cu at (79.9, 135.0)
- added R8: 10k, Resistor_SMD:R_0201_0603Metric, F.Cu at (79.9, 136.8)
- added U3: ESP32-WROOM-32, RF_Module:ESP32-WROOM-32, F.Cu at (66.5, 114.4)
- added U6: NRF24L01_Breakout, RF_Module:nRF24L01_Breakout, F.Cu at (44.7, 128.2)
- added U8: AP62150WU, Package_TO_SOT_SMD:TSOT-23-6, F.Cu at (88.3, 133.4)
- moved U2 125.8 mm to (258.9, 125.3), turned to 0 degrees
- moved R4 121.9 mm to (256.7, 122.1), turned to 0 degrees
- moved C5 119.2 mm to (254.2, 118.6), turned to 0 degrees
- moved C6 118.7 mm to (247.7, 122.8), turned to 0 degrees
- moved C1 118.5 mm to (251.8, 118.6), turned to 0 degrees
- moved C2 118.5 mm to (251.8, 120.4), turned to 0 degrees
- moved U5 117.7 mm to (253.1, 130.9), turned to 0 degrees
- moved R3 116.9 mm to (256.7, 120.4), turned to 0 degrees
- moved R2 115.0 mm to (256.7, 118.6), turned to 0 degrees
- moved C8 114.9 mm to (247.7, 129.5)
- moved R1 113.9 mm to (254.2, 122.1), turned to 0 degrees
- moved L1 111.5 mm to (253.6, 125.8), turned to 0 degrees
- moved C9 109.9 mm to (254.2, 120.4)
- moved C10 107.2 mm to (247.7, 132.8), turned to 0 degrees
- moved C7 104.7 mm to (247.7, 126.1), turned to 0 degrees
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Connections:
- net /IO18 renamed /Transmitter Side/IO18
- net /IO19 renamed /Transmitter Side/IO19
- net /IO22 renamed /Transmitter Side/IO22
- net /IO23 renamed /Transmitter Side/IO23
- net /IO25 renamed /Transmitter Side/IO25
- net /IO26 renamed /Transmitter Side/IO26
- net /IO27 renamed /Transmitter Side/IO27
Routing:
- net +3.3V: track 88.9 -> 0.00 mm, vias 3 -> 0
- net /Transmitter Side/IO23: track 54.1 -> 0.00 mm, vias 2 -> 0
- net /Transmitter Side/IO19: track 51.6 -> 0.00 mm, vias 2 -> 0
- net /Transmitter Side/IO18: track 47.3 -> 0.00 mm, vias 2 -> 0
- net /Transmitter Side/IO26: track 34.4 -> 0.00 mm
- net /Transmitter Side/IO25: track 30.9 -> 0.00 mm, vias 1 -> 0
- net /Transmitter Side/IO22: track 25.8 -> 0.00 mm, vias 1 -> 0
- net /Transmitter Side/IO27: track 9.68 -> 0.00 mm
- net Net-(U5-SW): track 6.80 -> 0.00 mm
- net Net-(U5-EN): track 4.62 -> 0.00 mm
- net Vin: track 2.99 -> 0.00 mm
- net Net-(U5-FB): track 2.16 -> 0.00 mm
- net Net-(U1-EN): track 1.63 -> 0.00 mm
- net Net-(U5-BST): track 1.39 -> 0.00 mm
- removed copper zone on F.Cu, net GND
