File: Temp Reader/Temp Reader.kicad_sch (KiCad schematic)
At the start: 1 part, among them U1 CDP1802BCE

Commit message: 1.First Commit
Save
Parts:
- removed U1: CDP1802BCE, Package_DIP:DIP-40_W15.24mm, symbol CPU:CDP1802BCE
- added U1: ESP32-WROOM-32, RF_Module:ESP32-WROOM-32, symbol RF_Module:ESP32-WROOM-32
- added U2: BME280, Package_LGA:Bosch_LGA-8_2.5x2.5mm_P0.65mm_ClockwisePinNumbering, symbol Sensor:BME280
- added U4: NRF24L01_Breakout, RF_Module:nRF24L01_Breakout, symbol RF:NRF24L01_Breakout
Connections:
- new net: U1.1 (GND), U1.15 (GND), U1.38 (GND), U1.39 (GND)
- new net CE: U1.10 (IO25)
- new net CSB: U1.12 (IO27)
- new net CSN: U1.36 (IO22)
- new net IO18: U2.4 (SCK), U4.5 (SCK)
- new net IO19: U2.5 (SDO), U4.7 (MISO)
- new net IO22: U4.4 (~{CSN})
- new net IO23: U2.3 (SDI), U4.6 (MOSI)
- new net IO25: U4.3 (CE)
- new net IO26: U4.8 (IRQ)
- new net IO27: U2.2 (CSB)
- new net IRQ: U1.11 (IO26)
- new net MISO: U1.31 (IO19)
- new net MOSI: U1.37 (IO23)
- new net SCK: U1.30 (IO18)

Commit message: 2.First Schematic Look
No Buck

Raw schematic
Parts:
- added C1, C2, C3, C5: 100nF, symbol Device:C_Small
- added C4, C6: 10uF, symbol Device:C_Small
Connections:
- net GND: now reaches U4.1 (GND)
- net GND: now also U1.1 (GND), U1.15 (GND), U1.38 (GND), U1.39 (GND), U2.1 (GND), U2.7 (GND), C1.1, C2.2, C3.2, C4.2, C5.2, C6.2
- net +3.3V: now reaches U4.2 (VCC)
- net +3.3V: now also U1.2 (VDD), U2.6 (VDDIO), U2.8 (VDD), C1.2, C2.1, C3.1, C4.1, C5.1, C6.1
- no-connect marks 0 -> 23
Other:
- note added: "ESP32 Capacitor Filter"
- note added: "NFR24L01 Capacitor Filter"
- moved on the sheet: U1, U2, U4

Commit message: 3. 80% schematic done
Parts:
- added C10, C7, C8: 22uF, symbol Device:C_Small
- added C9: 100nF, symbol Device:C_Small
- added L1: 2.2 uH, symbol Device:L
- added R1: 31.25k, symbol Device:R_Small
- added R2: 10k, symbol Device:R_Small
- added R3: 100k, symbol Device:R_Small
- added U5: AP62150WU, Package_TO_SOT_SMD:TSOT-23-6, symbol Regulator_Switching:AP62150WU
Connections:
- net GND: now also C10.2, C7.2, C8.2, R2.2, U5.1 (GND)
- new net: C9.1, U5.6 (BST)
- new net: C9.2, L1.1, U5.2 (SW)
- new net: R1.2, R2.1, U5.4 (FB)
- new net: R3.2, U5.5 (EN)
- new net Vin: C8.1, R3.1, U5.3 (VIN)
- new net Vout: C10.1, C7.1, L1.2, R1.1
Other:
- note added: "3.3V"
- note added: "6V"
- note added: "ANTENNA"
- note added: "BUCK 6V-3.3V"
- note added: "ESP32-THE BRAIN"
- note added: "WEATHER SENSOR"
- moved on the sheet: C1, C2, C3, C4, C5, C6, U1, U2, U4

Commit message: Allmost done , pcb start
Parts:
- added R4: 10k, symbol Device:R_Small
Connections:
- net CE is gone; now on net IO25: U1.10 (IO25)
- net CSB is gone; now on net IO27: U1.12 (IO27)
- net CSN is gone; now on net IO22: U1.36 (IO22)
- net IRQ is gone; now on net IO26: U1.11 (IO26)
- net MISO is gone; now on net IO19: U1.31 (IO19)
- net MOSI is gone; now on net IO23: U1.37 (IO23)
- net SCK is gone; now on net IO18: U1.30 (IO18)
- net +3.3V: now also R4.1
- net at U1.3 (EN): now also R4.2
- no-connect marks 23 -> 25
Other:
- note added: "TRANSMITTER SIDE"
- moved on the sheet: C5, C6, U1

Commit message: **First PCB , Not done yet
Parts:
- C1, C2, C3, C5, C9: footprint (none) -> Capacitor_SMD:C_0201_0603Metric
- C10, C4, C6, C7, C8: footprint (none) -> Capacitor_SMD:C_1206_3216Metric
- L1: footprint (none) -> Inductor_SMD:L_Bourns-SRN4018
- R1, R2, R3, R4: footprint (none) -> Resistor_SMD:R_0201_0603Metric
Connections:
- net Vout is gone; now on net +3.3V: C10.1, C7.1, L1.2, R1.1
Other:
- moved on the sheet: C10, C7, C8, C9, L1, R1, R2, R3, U5
